File: circuits/ethernet.sch (KiCad schematic (older format))
At the start: 28 parts, among them J12 RJ45_LED, Q8 Q_LMUN2211LT1G, U12 LAN8720A

Commit message: finished schematic corrections, working on layout
Parts:
- removed C19: C_1nF_1206, Capacitor_SMD:C_1206_3216Metric_Pad1.33x1.80mm_HandSolder, symbol Open_Automation:C_1nF_1206
- removed J12: RJ45_LED, Connector_RJ:RJ45_Abracon_ARJP11A-MA_Horizontal, symbol Open_Automation:RJ45_LED
- renumbered C20 to C29, C21 to C30, C22 to C31, C23 to C32, C24 to C33, C29 to C34, C25 to C35, C26 to C36, C27 to C37, C28 to C38, L3 to L2, Q8 to Q9, R53 to R67, R54 to R68, R55 to R69, R61 to R70, R56 to R71, R57 to R72, R58 to R73, R59 to R74, R60 to R75, R62 to R76, RM_2.2K2 to RM_2.2K1, U12 to U15
Connections:
- net labels added: MDCT1, MDCT2
- net labels removed: Earth, SP1, SP2
- wire segments 135 -> 127

Commit message: Disable Keypad when fob disarms lock. This is so the keypad does not rearm the lock if used.
Parts:
- C34: footprint Capacitor_SMD:C_0603_1608Metric_Pad1.08x0.95mm_HandSolder -> Capacitor_SMD:C_0805_2012Metric_Pad1.18x1.45mm_HandSolder; LCSC C96446 -> C15850; Part Number CL10A106MA8NRNC -> CL21A106KAYNNNE
- R74, R75: LCSC C1525 -> C25879; Part Number CL05B104KO5NNNC -> 0402WGF2201TCE
Changed lines of the file:
@@
 F 1 "R_2K2_0402" V 6000 3950 50  0000 L CNN
 F 2 "Resistor_SMD:R_0402_1005Metric_Pad0.72x0.64mm_HandSolder" V 5830 4150 50  0001 C CNN
-F 3 "https://datasheet.lcsc.com/szlcsc/Samsung-Electro-Mechanics-CL05B104KO5NNNC_C1525.pdf" V 5980 4150 50  0001 C CNN
-F 4 "CL05B104KO5NNNC" V 6080 4250 60  0001 C CNN "Part Number"
-F 5 "C1525" V 5750 4150 50  0001 C CNN "LCSC"
+F 3 "https://datasheet.lcsc.com/lcsc/1811022110_UNI-ROYAL-Uniroyal-Elec-0402WGF2201TCE_C25879.pdf" V 5980 4150 50  0001 C CNN
+F 4 "0402WGF2201TCE" V 6080 4250 60  0001 C CNN "Part Number"
+F 5 "C25879" V 5750 4150 50  0001 C CNN "LCSC"
 	1    5900 4150
 	1    0    0    -1
@@
 F 1 "R_2K2_0402" V 5850 1500 50  0000 L CNN
 F 2 "Resistor_SMD:R_0402_1005Metric_Pad0.72x0.64mm_HandSolder" V 5830 2100 50  0001 C CNN
-F 3 "https://datasheet.lcsc.com/szlcsc/Samsung-Electro-Mechanics-CL05B104KO5NNNC_C1525.pdf" V 5980 2100 50  0001 C CNN
-F 4 "CL05B104KO5NNNC" V 6080 2200 60  0001 C CNN "Part Number"
-F 5 "C1525" V 5750 2100 50  0001 C CNN "LCSC"
+F 3 "https://datasheet.lcsc.com/lcsc/1811022110_UNI-ROYAL-Uniroyal-Elec-0402WGF2201TCE_C25879.pdf" V 5980 2100 50  0001 C CNN
+F 4 "0402WGF2201TCE" V 6080 2200 60  0001 C CNN "Part Number"
+F 5 "C25879" V 5750 2100 50  0001 C CNN "LCSC"
 	1    5900 2100
 	1    0    0    -1
@@
 F 0 "C34" H 5950 6000 50  0000 C CNN
 F 1 "C_10uF" H 6000 6200 50  0000 C CNN
-F 2 "Capacitor_SMD:C_0603_1608Metric_Pad1.08x0.95mm_HandSolder" H 6300 6550 50  0001 C CNN
-F 3 "https://datasheet.lcsc.com/szlcsc/Samsung-Electro-Mechanics-CL10A106MA8NRNC_C96446.pdf" H 6050 5850 50  0001 C CNN
-F 4 "CL10A106MA8NRNC" H 6100 6650 60  0001 C CNN "Part Number"
-F 5 "C96446" H 6050 6750 50  0001 C CNN "LCSC"
+F 2 "Capacitor_SMD:C_0805_2012Metric_Pad1.18x1.45mm_HandSolder" H 6300 6550 50  0001 C CNN
+F 3 "https://datasheet.lcsc.com/szlcsc/Samsung-Electro-Mechanics-CL21A106KAYNNNE_C15850.pdf" H 6050 5850 50  0001 C CNN
+F 4 "CL21A106KAYNNNE" H 6100 6650 60  0001 C CNN "Part Number"
+F 5 "C15850" H 6050 6750 50  0001 C CNN "LCSC"
 	1    6050 6100
 	-1   0    0    1
