File: circuits/poe.sch (KiCad schematic (older format))
At the start: 44 parts, among them J19 Conn_02x02_Odd_Even, Q10 Q_FDC2512, Q11 Q_PNP_BEC, Q8 Q_FDC2512, U11 TPS23754PWP-1, U12 OPTO-FOD817A, U13 TLV431ACDBZR

Commit message: Disable Keypad when fob disarms lock. This is so the keypad does not rearm the lock if used.
Parts:
- C17: footprint Capacitor_SMD:C_1206_3216Metric_Pad1.33x1.80mm_HandSolder -> Capacitor_SMD:C_0603_1608Metric_Pad1.08x0.95mm_HandSolder; LCSC C16772 -> C21120; Part Number CL05B224KO5NNNC -> CL10B224KA8NNNC
- R47, R48: footprint Resistor_SMD:R_0603_1608Metric_Pad0.98x0.95mm_HandSolder -> Resistor_SMD:R_0402_1005Metric_Pad0.72x0.64mm_HandSolder
Connections:
- net at D12.2 (NC): now also R61.2
Changed lines of the file:
@@
 F 0 "R47" V 850 3650 50  0000 C CNN
 F 1 "R_3.01K" V 950 3700 50  0000 C CNN
-F 2 "Resistor_SMD:R_0603_1608Metric_Pad0.98x0.95mm_HandSolder" V 780 3650 50  0001 C CNN
+F 2 "Resistor_SMD:R_0402_1005Metric_Pad0.72x0.64mm_HandSolder" V 780 3650 50  0001 C CNN
 F 3 "https://datasheet.lcsc.com/szlcsc/Uniroyal-Elec-0402WGF3011TCE_C25889.pdf" V 930 3650 50  0001 C CNN
 F 4 "0402WGF3011TCE" V 1030 3750 60  0001 C CNN "Part Number"
@@
 F 0 "R48" V 1050 3500 50  0000 C CNN
 F 1 "R_69.8K" V 1150 3550 50  0000 C CNN
-F 2 "Resistor_SMD:R_0603_1608Metric_Pad0.98x0.95mm_HandSolder" V 980 3500 50  0001 C CNN
+F 2 "Resistor_SMD:R_0402_1005Metric_Pad0.72x0.64mm_HandSolder" V 980 3500 50  0001 C CNN
 F 3 "https://datasheet.lcsc.com/szlcsc/Uniroyal-Elec-0402WGF6982TCE_C26985.pdf" V 1130 3500 50  0001 C CNN
 F 4 "0402WGF6982TCE" V 1230 3600 60  0001 C CNN "Part Number"
@@
 F 0 "C17" H 3000 5600 50  0000 L CNN
 F 1 "C_220nF" H 2850 5400 50  0000 L CNN
-F 2 "Capacitor_SMD:C_1206_3216Metric_Pad1.33x1.80mm_HandSolder" H 3300 5800 50  0001 C CNN
-F 3 "https://datasheet.lcsc.com/szlcsc/Samsung-Electro-Mechanics-CL05B224KO5NNNC_C16772.pdf" H 3200 5250 50  0001 C CNN
-F 4 "C16772" H 3200 5900 50  0001 C CNN "LCSC"
-F 5 "CL05B224KO5NNNC" H 3325 5700 60  0001 C CNN "Part Number"
+F 2 "Capacitor_SMD:C_0603_1608Metric_Pad1.08x0.95mm_HandSolder" H 3300 5800 50  0001 C CNN
+F 3 "https://datasheet.lcsc.com/szlcsc/Samsung-Electro-Mechanics-CL10B224KA8NNNC_C21120.pdf" H 3200 5250 50  0001 C CNN
+F 4 "C21120" H 3200 5900 50  0001 C CNN "LCSC"
+F 5 "CL10B224KA8NNNC" H 3325 5700 60  0001 C CNN "Part Number"
 	1    3200 5500
 	1    0    0    -1
