File: circuits/controller/control.kicad_sch (KiCad schematic)
At the start: 8 parts, among them Q1 Q_MMBT5551, Q2 Q_AO3400A, Q3 Q_MMBT5551, Q4 Q_AO3400A

Commit message: sent to fab! 0.6
Parts:
- renumbered Q1 to Q6, Q3 to Q7, Q2 to Q8, Q4 to Q9, R4 to R53, R5 to R54, R6 to R55, R7 to R56
