File: circuits/controller/quad-optocoupler.kicad_sch (KiCad schematic)
At the start: 9 parts, among them U3 TLP291-4

Commit message: sent to fab! 0.6
Parts:
- renumbered R8 to R16, R9 to R17, R10 to R18, R11 to R19, U3 to U5
Connections:
- net TRIGGER0: now also R12.2; no longer R15.2
- net TRIGGER1: now also R13.2; no longer R12.2
- net TRIGGER2: now also R14.2; no longer R13.2
- net TRIGGER3: now also R15.2; no longer R14.2
Changed lines of the file:
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@@
-(kicad_sch (version 20211123) (generator eeschema)
+(kicad_sch (version 20230121) (generator eeschema)
   (paper "A4")
