File: circuits/controller/usb.kicad_sch (KiCad schematic)
At the start: 16 parts, among them J18 USB_MINI_B, Q5 Crystal_12Mhz, Q6 Q_SS8050, Q7 Q_SS8550, U10 CH340T(SSOP20W)

Commit message: sent to fab! 0.6
Parts:
- renumbered C7 to C16, C8 to C17, C9 to C18, C10 to C19, D7 to D13, J18 to J22, Q5 to Q3, Q6 to Q4, Q7 to Q5, R41 to R31, R42 to R32, R43 to R33, R44 to R34, R45 to R35, R46 to R36, U10 to U8
