File: circuits/controller/wiegand.kicad_sch (KiCad schematic)
At the start: 16 parts, among them Q10 Q_MMBT5551, Q11 Q_MMBT5551, Q12 Q_MMBT5551, Q13 Q_MMBT5551, Q14 Q_MMBT5551, Q8 Q_MMBT5551

Commit message: sent to fab! 0.6
Parts:
- renumbered Q8 to Q10, Q10 to Q11, Q11 to Q12, Q12 to Q13, Q13 to Q14, Q14 to Q15, R20 to R57, R21 to R58, R34 to R59, R37 to R60, R40 to R61, R47 to R62, R48 to R63, R49 to R64, R50 to R65, R51 to R66
