File: circuits/controller/microcontroller.kicad_sch (KiCad schematic)
At the start: 12 parts, among them U14 ESP32-WROOM-32

Commit message: sent to fab! 0.6
Parts:
- removed C26: C_10uF, Capacitor_SMD:C_0805_2012Metric_Pad1.18x1.45mm_HandSolder, symbol Open_Automation:C_10uF
- removed C27: C_1uF, Capacitor_SMD:C_0402_1005Metric_Pad0.74x0.62mm_HandSolder, symbol Open_Automation:C_1uF
- removed D16, D17, D18: LED_G, LED_SMD:LED_0603_1608Metric_Pad1.05x0.95mm_HandSolder, symbol Open_Automation:LED_G
- removed EN1, FACT1, PROG1: SW_PUSH, Button_Switch_SMD:SW_SPST_PTS645, symbol Open_Automation:SW_PUSH
- removed R64, R65, R66: 10K, Resistor_SMD:R_0402_1005Metric_Pad0.72x0.64mm_HandSolder, symbol Open Automation:R_10K_0402
- removed U14: ESP32-WROOM-32, RF_Module:ESP32-WROOM-32, symbol Open_Automation:ESP32-WROOM-32
- added C40, C41: C_10uF, Capacitor_SMD:C_0805_2012Metric_Pad1.18x1.45mm_HandSolder, symbol open_automation:C_10uF
- added C42: 100nF, Capacitor_SMD:C_0402_1005Metric_Pad0.74x0.62mm_HandSolder, symbol open_automation:C_100nF_0402
- added C43, C44: 1uF, Capacitor_SMD:C_0402_1005Metric_Pad0.74x0.62mm_HandSolder, symbol open_automation:C_1uF
- added C47: 1uF, Capacitor_SMD:C_0402_1005Metric_Pad0.74x0.62mm_HandSolder, symbol Open_Automation:C_1uF
- added C48: C_10uF, Capacitor_SMD:C_0805_2012Metric_Pad1.18x1.45mm_HandSolder, symbol Open_Automation:C_10uF
- added D10, D11, D12, D14, D15, D17: ESD_5V, Diode_SMD:D_SOD-523, symbol open_automation:D_ESD9B5.0ST5G
- added D13, D16: D_1N5819HW, Diode_SMD:D_SOD-123, symbol open_automation:D_1N5819HW
- added EN1, FACT1, PROG1: SW_PUSH, Button_Switch_SMD:SW_SPST_PTS645, symbol open-dash-daughterboard-rescue:SW_PUSH-Open_Automation
- added J8, J9: USB_MINI_B, Connector_USB:USB_Mini-B_Wuerth_65100516121_Horizontal, symbol open_automation:USB_MINI_B_SMD
- added Q1: Q_L8050QLT1G, Package_TO_SOT_SMD:SOT-23, symbol open_automation:Q_L8050QLT1G
- added Q2: Q_L8550HQLT1G, Package_TO_SOT_SMD:SOT-23, symbol open_automation:Q_L8550HQLT1G
- added R30, R31, R32, R33, R34, R38, R39, R40: 10K, Resistor_SMD:R_0402_1005Metric_Pad0.72x0.64mm_HandSolder, symbol Open_Automation:R_10K_0402
- added R35: 22.1K, Resistor_SMD:R_0402_1005Metric_Pad0.72x0.64mm_HandSolder, symbol open_automation:R_22.1K_0402
- added R36: 47.5K, Resistor_SMD:R_0603_1608Metric_Pad0.98x0.95mm_HandSolder, symbol open_automation:R_47.5k
- added R37: 1K, Resistor_SMD:R_0402_1005Metric_Pad0.72x0.64mm_HandSolder, symbol open_automation:R_1K_0402
- added U1: CP2102N-Axx-xQFN28, Package_DFN_QFN:QFN-28-1EP_5x5mm_P0.5mm_EP3.35x3.35mm, symbol Interface_USB:CP2102N-Axx-xQFN28
- added U3: ESP32-S3-WROOM-1, Espressif:ESP32-S3-WROOM-1, symbol Espressif:ESP32-S3-WROOM-1
Connections:
- net 3V3: now also C42.1, C48.1, R32.1, R33.1, R34.1, R37.1, R39.1, R40.2, U1.6 (VDD), U1.7 (VREGIN), U3.2 (3V3)
- net FACT: now also FACT1.1, R32.2, U3.39 (GPIO1/TOUCH1/ADC1_CH0)
- net GND: now also C40.2, C41.2, C42.2, C43.2, C44.2, C47.2, C48.2, D10.1 (A1), D11.1 (A1), D12.1 (A1), D14.1 (A1), D15.1 (A1), D17.1 (A1), EN1.2, FACT1.2, J8.5 (GND), J9.5 (GND), PROG1.2, R36.1, R38.2, U1.29 (GND), U1.3 (GND), U3.1 (GND), U3.40 (GND), U3.41 (GND)
- net IO12: now also U3.20 (GPIO12/TOUCH12/ADC2_CH1/FSPICLK/FSPIIO6/SUBSPICLK)
- net IO15: now also U3.8 (GPIO15/U0RTS/ADC2_CH4/XTAL_32K_P)
- net IO16: now also U3.9 (GPIO16/U0CTS/ADC2_CH5/XTAL_32K_N)
- net IO17: now also U3.10 (GPIO17/U1TXD/ADC2_CH6)
- net IO18: now also U3.11 (GPIO18/U1RXD/ADC2_CH7/CLK_OUT3)
- net IO19: now also D15.2 (A2), J9.2 (D-), U3.13 (GPIO19/U1RTS/ADC2_CH8/CLK_OUT2/USB_D-)
- net IO2: now also U3.38 (GPIO2/TOUCH2/ADC1_CH1)
- net IO21: now also U3.23 (GPIO21)
- net IO35: now also U3.28 (SPIIO6/GPIO35/FSPID/SUBSPID)
- net IO4: now also U3.4 (GPIO4/TOUCH4/ADC1_CH3)
- net IO5: now also U3.5 (GPIO5/TOUCH5/ADC1_CH4)
- net PROG: now also C47.1, PROG1.1, Q2.2 (E), R33.2, U3.27 (GPIO0/BOOT)
- new net: C44.1, R35.1, R36.2, U1.8 (VBUS)
- new net: D16.2 (A), J9.1 (VBUS)
- new net: R37.2, U1.9 (~{RST})
- new net: R38.1, U1.11 (~{SUSPEND})
- new net: Q1.1 (B), R30.2
- new net: D13.2 (A), J8.1 (VBUS)
- new net: Q2.1 (B), R31.2
- new net 5V: C40.1, C41.1, D12.2 (A2), D13.1 (K), D16.1 (K), D17.2 (A2), R35.2
- new net D+: D11.2 (A2), J8.3 (D+), U1.4 (D+)
- new net D-: D10.2 (A2), J8.2 (D-), U1.5 (D-)
- new net DTR: Q2.3 (C), R30.1, U1.28 (~{DTR})
- new net EN: C43.1, EN1.1, Q1.3 (C), R34.2, U3.3 (EN)
- new net I2C_CLK: R40.1, U3.21 (GPIO13/TOUCH13/ADC2_CH2/FSPIQ/FSPIIO7/SUBSPIQ)
- new net I2C_DATA: R39.2, U3.22 (GPIO14/TOUCH14/ADC2_CH3/FSPIWP/FSPIDQS/SUBSPIWP)
- new net IO10: U3.18 (GPIO10/TOUCH10/ADC1_CH9/FSPICS0/FSPIIO4/SUBSPICS0)
- new net IO11: U3.19 (GPIO11/TOUCH11/ADC2_CH0/FSPID/FSPIIO5/SUBSPID)
- new net IO20: D14.2 (A2), J9.3 (D+), U3.14 (GPIO20/U1CTS/ADC2_CH9/CLK_OUT1/USB_D+)
- new net IO3: U3.15 (GPIO3/TOUCH3/ADC1_CH2)
- new net IO36: U3.29 (SPIIO7/GPIO36/FSPICLK/SUBSPICLK)
- new net IO37: U3.30 (SPIDQS/GPIO37/FSPIQ/SUBSPIQ)
- new net IO38: U3.31 (GPIO38/FSPIWP/SUBSPIWP)
- new net IO39: U3.32 (MTCK/GPIO39/CLK_OUT3/SUBSPICS1)
- new net IO40: U3.33 (MTDO/GPIO40/CLK_OUT2)
- new net IO41: U3.34 (MTDI/GPIO41/CLK_OUT1)
- new net IO42: U3.35 (MTMS/GPIO42)
- new net IO43: U1.25 (RXD), U3.37 (U0TXD/GPIO43/CLK_OUT1)
- new net IO44: U1.26 (TXD), U3.36 (U0RXD/GPIO44/CLK_OUT2)
- new net IO45: U3.26 (GPIO45)
- new net IO46: U3.16 (GPIO46)
- new net IO47: U3.24 (GPIO47/SPICLK_P/SUBSPICLK_P_DIFF)
- new net IO48: U3.25 (GPIO48/SPICLK_N/SUBSPICLK_N_DIFF)
- new net IO6: U3.6 (GPIO6/TOUCH6/ADC1_CH5)
- new net IO7: U3.7 (GPIO7/TOUCH7/ADC1_CH6)
- new net IO8: U3.12 (GPIO8/TOUCH8/ADC1_CH7/SUBSPICS1)
- new net IO9: U3.17 (GPIO9/TOUCH9/ADC1_CH8/FSPIHD/SUBSPIHD)
- new net RTS: Q1.2 (E), R31.1, U1.24 (~{RTS})
- no-connect marks 7 -> 15

Commit message: order from fab
Changed lines of the file:
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@@
+    (stroke (width 0) (type default))
+  )
+  (wire (pts (xy 68.58 86.233) (xy 69.85 86.233))
     (stroke (width 0) (type default))
   )
@@
     (stroke (width 0) (type default))
   )
+  (wire (pts (xy 68.58 83.82) (xy 69.85 83.82))
+    (stroke (width 0) (type default))
+  )
   (wire (pts (xy 319.7606 182.7784) (xy 295.8846 182.7784))
     (stroke (width 0) (type default))
@@
     (effects (font (size 1.27 1.27)) (justify left bottom))
   )
+  (label "IO15" (at 69.85 83.82 0) (fields_autoplaced)
+    (effects (font (size 1.27 1.27)) (justify left bottom))
+  )
   (label "PROG" (at 320.1416 205.0034 0) (fields_autoplaced)
     (effects (font (size 1.27 1.27)) (justify left bottom))
@@
     (effects (font (size 1.27 1.27)) (justify left bottom))
   )
+  (label "IO16" (at 69.85 86.233 0) (fields_autoplaced)
+    (effects (font (size 1.27 1.27)) (justify left bottom))
+  )
   (label "IO40" (at 227.0506 78.5114 180) (fields_autoplaced)
     (effects (font (size 1.27 1.27)) (justify right bottom))
@@
     (effects (font (size 1.524 1.524)) (justify right))
   )
+  (hierarchical_label "IO16" (shape input) (at 68.58 86.233 180) (fields_autoplaced)
+    (effects (font (size 1.524 1.524)) (justify right))
+  )
   (hierarchical_label "I2C_CLK" (shape input) (at 65.5066 60.4774 180) (fields_autoplaced)
     (effects (font (size 1.524 1.524)) (justify right))
   )
+  (hierarchical_label "IO15" (shape input) (at 68.58 83.82 180) (fields_autoplaced)
+    (effects (font (size 1.524 1.524)) (justify right))
+  )
